File: _autosave-m3++.kicad_pcb (KiCad board)
At the start: 2 copper layers, 102 x 122 mm, 17 parts, among them SW1 SW_Push, SW10 SW_Push, SW11 SW_Push, SW12 SW_Push, SW2 SW_Push, SW3 SW_Push, SW4 SW_Push, SW5 SW_Push, SW6 SW_Push, SW7 SW_Push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

Commit message: initial commit
Other:
- board text added: "docking takes place at home. yiffing takes place on your own time."
Changed lines of the file:
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@@
 			)
 		)
-		(fp_text user "Ethernet"
+		(fp_text user "aoifernet"
 			(at -12.065 -3.2766 0)
 			(layer "F.SilkS")
@@
 				(font
 					(size 1 1)
-					(thickness 0.15)
-				)
-			)
-		)
-		(fp_text user "DVJ6A"
-			(at -2.54 -0.18 0)
-			(layer "F.SilkS")
-			(effects
-				(font
-					(size 0.7 0.7)
 					(thickness 0.15)
 				)
@@
 				(font
 					(size 1 1)
-					(thickness 0.15)
-				)
-			)
-		)
-		(fp_text user "MIMXRT1062"
-			(at -1.27 0 0)
-			(layer "F.SilkS")
-			(effects
-				(font
-					(size 0.7 0.7)
 					(thickness 0.15)
 				)
@@
 		(layer "Edge.Cuts")
 	)
+	(gr_text "docking takes place at home.\nyiffing takes place on your own time."
+		(at 189 125.5 0)
+		(layer "B.SilkS")
+		(effects
+			(font
+				(size 1 1)
+				(thickness 0.1)
+			)
+			(justify left bottom mirror)
+		)
+	)
 	(gr_text "mounting takes place here"
