File: kicad/m3++.kicad_pcb (KiCad board)
At the start: 2 copper layers, 102 x 122 mm, 17 parts, among them SW1 SW_Push, SW10 SW_Push, SW11 SW_Push, SW12 SW_Push, SW2 SW_Push, SW3 SW_Push, SW4 SW_Push, SW5 SW_Push, SW6 SW_Push, SW7 SW_Push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

Commit message: finished pcb design
design files when ordered
Other:
- board text added: "HERE"
- board text added: "and emptier..."
- board text added: "hytheaway 2024 ^-^ https://hytheaway.github.io"
- board text added: "i will break"
- board text added: "if you snap me"
- board text added: "kirby"
- board text added: "look at all these traces :o"
- board text added: "make sure you step over them!"
- board text added: "olimar"
- board text added: "pikachu"
- board text added: "the space gets emptier..."
- board text added: "this bridge is provided ->"
- board text added: "this is a bunch of empty space."
- board text added: "this is the backside, btw"
- board text added: "this project is open. find it at https://github.com/hytheaway/m3--"
- board text removed: "hytheaway 2024 ^-^"
